Commit message: added new untested urdf model with dovetail

File: xacro/gummi_description_ee.urdf.xacro (robot description, xacro)
@@ -1,66 +1,102 @@
 <?xml version="1.0" encoding="utf-8"?>
-  <!-- j5_Link -->
-  <robot>
-    <link name="lowerarm_preroll_d">
-        <visual>
-        <origin xyz="0.084 0 -0.012" rpy="0 0 0" />
-        <geometry>
-          <box size=".02 .05 .05" />
-        </geometry>
-        <material name="not Cyan">
-          <color rgba="1 0.7 0.7 1"/>
-        </material>
-      </visual>
-      </link>
-      <joint name="fastswitch" type="fixed">
-        <origin rpy="0 0 0" xyz="0.00 -0.015 0"/>
-        <parent link="lowerarm_preroll_u"/>
-        <child link="lowerarm_preroll_d"/>
-      </joint>
-  <!-- j6_Link -->
+<robot>
+  <link
+    name="lowerarm_preroll_d">
+    <inertial>
+      <origin
+        xyz="0.0192090313803226 -0.000209732444885397 -0.00477606520095217"
+        rpy="0 0 0" />
+      <mass
+        value="0.0573922743530686" />
+      <inertia
+        ixx="5.98272304285402E-07"
+        ixy="-9.55132100709239E-09"
+        ixz="2.00959509125472E-06"
+        iyy="7.34863588332809E-06"
+        iyz="2.84343934345717E-09"
+        izz="6.7503906079721E-06" />
+    </inertial>
+    <visual>
+      <origin
+        xyz="0 0 0"
+        rpy="0 0 0" />
+      <geometry>
+        <mesh
+          filename="package://gummi_ee_$(env ROS_GUMMI_EE)/meshes/lowerarm_preroll_d.STL" />
+      </geometry>
+      <material
+        name="">
+        <color
+          rgba="0.792156862745098 0.819607843137255 0.933333333333333 1" />
+      </material>
+    </visual>
+    <collision>
+      <origin
+        xyz="0 0 0"
+        rpy="0 0 0" />
+      <geometry>
+        <mesh
+          filename="package://gummi_ee_$(env ROS_GUMMI_EE)/meshes/lowerarm_preroll_d.STL" />
+      </geometry>
+    </collision>
+  </link>
+  <joint
+    name="fastswitch"
+    type="fixed">
+    <origin
+      xyz="0.056236 -0.019 -0.006"
+      rpy="0 0 0" />
+    <parent
+      link="lowerarm_preroll_u" />
+    <child
+      link="lowerarm_preroll_d" />
+    <axis
+      xyz="0 0 0" />
+  </joint>
   <link
     name="lowerarm">
     <inertial>
       <origin
-        xyz="0.063088 -4.524E-06 0.010537"
-        rpy="0 0 0" />
-      <mass
-        value="0.088554" />
-      <inertia
-        ixx="3.269E-05"
-        ixy="2.0124E-07"
-        ixz="-1.6433E-05"
-        iyy="7.2394E-05"
-        iyz="1.982E-07"
-        izz="6.9913E-05" />
-    </inertial>
-    <visual>
-      <origin
-        xyz="0.09 0 0.01"
-        rpy="0 0 0" />
-      <geometry>
-        <box size=".16 .033 .052" />
-      </geometry>
-      <material
-        name="">
-        <color
-          rgba="0.79216 0.81961 0.93333 1" />
-      </material>
-    </visual>
-    <collision>
-      <origin
-        xyz="0.09 0 0.01"
-        rpy="0 0 0" />
-      <geometry>
-        <box size=".16 .033 .052" />
-      </geometry>
-    </collision>
-  </link>
-  <!-- j6 -->
+        xyz="0.076518166900465 0.000154587846369382 0.00668942647768447"
+        rpy="0 0 0" />
+      <mass
+        value="0.214658222402075" />
+      <inertia
+        ixx="2.53797627665925E-05"
+        ixy="-3.78406001691015E-09"
+        ixz="1.36269412886066E-05"
+        iyy="0.000325304336296306"
+        iyz="3.75496083335353E-07"
+        izz="0.000302080494837117" />
+    </inertial>
+    <visual>
+      <origin
+        xyz="0 0 0"
+        rpy="0 0 0" />
+      <geometry>
+        <mesh
+          filename="package://gummi_ee_$(env ROS_GUMMI_EE)/meshes/lowerarm.STL" />
+      </geometry>
+      <material
+        name="">
+        <color
+          rgba="0.792156862745098 0.819607843137255 0.933333333333333 1" />
+      </material>
+    </visual>
+    <collision>
+      <origin
+        xyz="0 0 0"
+        rpy="0 0 0" />
+      <geometry>
+        <mesh
+          filename="package://gummi_ee_$(env ROS_GUMMI_EE)/meshes/lowerarm.STL" />
+      </geometry>
+    </collision>
+  </link>
   <joint
     name="forearm_roll"
-    type="revolute">
-    <origin
-      xyz="0.0795 0.00025 -0.025"
+    type="continuous">
+    <origin
+      xyz="0.043506 -0.00023376 -0.019876"
       rpy="0 0 0" />
     <parent
@@ -69,57 +105,54 @@
       link="lowerarm" />
     <axis
-      xyz="1 0 0" />
-    <!-- <limit
-      lower="-1.5708"
-      upper="1.5708"
-      effort="0"
-      velocity="0" /> -->
-    <limit effort="0" lower="-2.7489" upper="2.7489" velocity="1.0"/>
-  </joint>
-  <!-- j7_Link -->
+      xyz="-1 0 0" />
+    <limit
+      effort="0"
+      velocity="1" />
+  </joint>
   <link
     name="wrist">
     <inertial>
       <origin
-        xyz="0.09547 -0.0036816 -0.028022"
-        rpy="0 0 0" />
-      <mass
-        value="0.20597" />
-      <inertia
-        ixx="0.00034354"
-        ixy="1.9986E-06"
-        ixz="3.1921E-05"
-        iyy="0.00045939"
-        iyz="2.5997E-08"
-        izz="0.00046029" />
-    </inertial>
-    <visual>
-      <origin
-        xyz="0.073 0 0"
-        rpy="0 0 0" />
-      <geometry>
-        <box size=".146 .06 .015" />
-      </geometry>
-      <material
-        name="">
-        <color
-          rgba="0.79216 0.81961 0.93333 1" />
-      </material>
-    </visual>
-    <collision>
-      <origin
-        xyz="0.073 0 0"
-        rpy="0 0 0" />
-      <geometry>
-        <box size=".146 .06 .015" />
-      </geometry>
-    </collision>
-  </link>
-  <!-- j7 -->
+        xyz="0.0484512742480244 0.0139768664666073 0.000956995637939325"
+        rpy="0 0 0" />
+      <mass
+        value="0.0644774651698934" />
+      <inertia
+        ixx="8.67406414845019E-06"
+        ixy="-1.3193756197629E-05"
+        ixz="-3.41916035169704E-06"
+        iyy="4.217442276821E-05"
+        iyz="-4.04257224014858E-07"
+        izz="4.91399139463636E-05" />
+    </inertial>
+    <visual>
+      <origin
+        xyz="0 0 0"
+        rpy="0 0 0" />
+      <geometry>
+        <mesh
+          filename="package://gummi_ee_$(env ROS_GUMMI_EE)/meshes/wrist.STL" />
+      </geometry>
+      <material
+        name="">
+        <color
+          rgba="0.792156862745098 0.819607843137255 0.933333333333333 1" />
+      </material>
+    </visual>
+    <collision>
+      <origin
+        xyz="0 0 0"
+        rpy="0 0 0" />
+      <geometry>
+        <mesh
+          filename="package://gummi_ee_$(env ROS_GUMMI_EE)/meshes/wrist.STL" />
+      </geometry>
+    </collision>
+  </link>
   <joint
     name="wrist_pitch"
     type="revolute">
     <origin
-      xyz="0.15 0 0.009003"
+      xyz="0.1511 -0.01935 0.0048471"
       rpy="0 0 0" />
     <parent
@@ -129,83 +162,299 @@
     <axis
       xyz="0 1 0" />
-      <!-- <limit
-        lower="-1.5708"
-        upper="1.5708"
-        effort="0"
-        velocity="0" /> -->
-      <limit effort="0" lower="-1.5" upper="1.68" velocity="1.0"/>
-  </joint>
-  <!-- gripper_Link -->
-  <link
-    name="gripper_Link">
-    <inertial>
-      <origin
-        xyz="-0.0233988267408998 -0.0183769778598925 -0.00217479089040148"
-        rpy="0 0 0" />
-      <mass
-        value="0.0573612129510164" />
-      <inertia
-        ixx="1.07017574054092E-05"
-        ixy="1.20541476778111E-07"
-        ixz="-2.08068523476524E-06"
-        iyy="6.40757036666839E-05"
-        iyz="3.89770387703761E-08"
-        izz="6.62562645856636E-05" />
-    </inertial>
-    <visual>
-      <origin
-        xyz="0.05 0 0"
-        rpy="0 0 0" />
-      <geometry>
-        <box size=".07 .008 .06" />
-      </geometry>
-      <material
-        name="">
-        <color
-          rgba="0.79216 0.81961 0.93333 1" />
-      </material>
-    </visual>
-    <collision>
-      <origin
-        xyz="0.05 0 0"
-        rpy="0 0 0" />
-      <geometry>
-        <box size=".07 .008 .06" />
-      </geometry>
-    </collision>
-  </link>
-  <!-- gripper -->
-  <joint
-    name="gripper"
-    type="revolute">
-    <origin
-      xyz="0.14 0 0"
-      rpy="1.5708 1.0472 3.1416" />
-    <parent
-      link="wrist" />
-    <child
-      link="gripper_Link" />
-    <axis
-      xyz="0 0 1" />
-    <!-- <limit
-      lower="-1.5708"
-      upper="1.5708"
-      effort="0"
-      velocity="0" /> -->
-    <limit effort="0" lower="-2.0" upper="0.37" velocity="1.0"/>
-  </joint>
-  <link name="tool">
-  </link>
-  <joint name="coupling_tool" type="fixed">
-    <origin rpy="0 0 0" xyz="0.175 -0.02 0.13"/>
-    <parent link="wrist"/>
-    <child link="tool"/>
-    <axis xyz="0 1 0"/>
-    <!-- <limit
-    lower="-1.5708"
-    upper="1.5708"
-    effort="0"
-    velocity="0" /> -->
-    <limit effort="0" lower="-0.30" upper="0.17" velocity="1.0"/>
+    <limit
+      lower="-1"
+      upper="1"
+      effort="0"
+      velocity="0" />
+  </joint>
+  <link
+    name="i1">
+    <inertial>
+      <origin
+        xyz="0.0230748926267925 0.00588066789200992 0.00129219082652174"
+        rpy="0 0 0" />
+      <mass
+        value="0.00632408233084942" />
+      <inertia
+        ixx="3.56498343502738E-08"
+        ixy="-7.51978011656011E-09"
+        ixz="7.65091950170785E-08"
+        iyy="1.38099634070148E-06"
+        iyz="2.95085409823962E-09"
+        izz="1.34584197546666E-06" />
+    </inertial>
+    <visual>
+      <origin
+        xyz="0 0 0"
+        rpy="0 0 0" />
+      <geometry>
+        <mesh
+          filename="package://gummi_ee_$(env ROS_GUMMI_EE)/meshes/i1.STL" />
+      </geometry>
+      <material
+        name="">
+        <color
+          rgba="0.792156862745098 0.819607843137255 0.933333333333333 1" />
+      </material>
+    </visual>
+    <collision>
+      <origin
+        xyz="0 0 0"
+        rpy="0 0 0" />
+      <geometry>
+        <mesh
+          filename="package://gummi_ee_$(env ROS_GUMMI_EE)/meshes/i1.STL" />
+      </geometry>
+    </collision>
+  </link>
+  <joint
+    name="i1f"
+    type="revolute">
+    <origin
+      xyz="0.059922 -0.031986 0.0029515"
+      rpy="-0.79367 0.12795 -0.91441" />
+    <parent
+      link="wrist" />
+    <child
+      link="i1" />
+    <axis
+      xyz="0 -1 0" />
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
File: xacro/gummi_ee.srdf.xacro (robot description, xacro)
@@ -2,17 +2,18 @@
 <robot name="gummi" xmlns:xacro="http://www.ros.org/wiki/xacro">
 <xacro:macro name="group_right_arm_ee">
-    <joint name="elbow" />
     <joint name="forearm_roll" />
     <joint name="wrist_pitch" />
-    <joint name="coupling_tool"/>
 </xacro:macro>
 <xacro:macro name="group_right_gripper_ee">
   <group name="right_gripper">
-      <link name="wrist" />
-      <link name="gripper_Link" />
+    <link name="wrist"/>
+    <joint name="i1f"/>
+    <joint name="i2f"/>
+    <joint name="i3f"/>
+    <joint name="i4f"/>
+    <joint name="i5f"/>
   </group>
 </xacro:macro>
 <xacro:macro name="group_state_right_arm_ee">
-  <joint name="elbow" value="0" />
   <joint name="forearm_roll" value="0" />
   <joint name="wrist_pitch" value="0" />
@@ -20,12 +21,29 @@
 <xacro:macro name="end_effector_ee">
   <!--END EFFECTOR: Purpose: Represent information about an end effector.-->
-<end_effector group="right_arm" name="right_eef" parent_link="tool"/>
+<end_effector group="right_gripper" name="right_eef" parent_link="wrist" parent_group="right_arm"/>
 </xacro:macro>
 <xacro:macro name="disable_collisions_ee">
   <!-- <disable_collisions link1="right_hand" link2="wrist" reason="Never" />
-  <disable_collisions link1="right_hand" link2="gripper_Link" reason="Never" /> -->
-  <disable_collisions link1="gripper_Link" link2="lowerarm" reason="Never" />
-  <disable_collisions link1="gripper_Link" link2="lowerarm_preroll_d" reason="Never" />
-  <disable_collisions link1="gripper_Link" link2="wrist" reason="Adjacent" />
+  <disable_collisions link1="right_hand" link2="gripper_link" reason="Never" /> -->
+  <disable_collisions link1="i1" link2="lowerarm" reason="Never" />
+  <disable_collisions link1="i2" link2="lowerarm" reason="Never" />
+  <disable_collisions link1="i3" link2="lowerarm" reason="Never" />
+  <disable_collisions link1="i4" link2="lowerarm" reason="Never" />
+  <disable_collisions link1="i5" link2="lowerarm" reason="Never" />
+  <disable_collisions link1="i1" link2="wrist" reason="Never" />
+  <disable_collisions link1="i2" link2="wrist" reason="Never" />
+  <disable_collisions link1="i3" link2="wrist" reason="Never" />
+  <disable_collisions link1="i4" link2="wrist" reason="Never" />
+  <disable_collisions link1="i5" link2="wrist" reason="Never" />
+  <disable_collisions link1="i1" link2="i2" reason="Never" />
+  <disable_collisions link1="i1" link2="i3" reason="Never" />
+  <disable_collisions link1="i1" link2="i4" reason="Never" />
+  <disable_collisions link1="i1" link2="i5" reason="Never" />
+  <disable_collisions link1="i2" link2="i3" reason="Never" />
+  <disable_collisions link1="i2" link2="i4" reason="Never" />
+  <disable_collisions link1="i2" link2="i5" reason="Never" />
+  <disable_collisions link1="i3" link2="i4" reason="Never" />
+  <disable_collisions link1="i3" link2="i5" reason="Never" />
+  <disable_collisions link1="i4" link2="i5" reason="Never" />
   <disable_collisions link1="lowerarm" link2="lowerarm_preroll_d" reason="Adjacent" />
   <disable_collisions link1="lowerarm" link2="wrist" reason="Adjacent" />

Commit message: added mimic to move finger joints appropriately and fixed srdf so it can move

File: xacro/gummi_description_ee.urdf.xacro (robot description, xacro)
@@ -168,4 +168,17 @@
       velocity="0" />
   </joint>
+  <!--
+  making sure I can move my fingers in a synchronized way. also if they move at
+  different rates, set the mimic tag to something different. it allows for an
+  offset and a multiplication rate. check ros docs for details
+  -->
+  <joint name="gripper" type="revolute">
+    <origin rpy="0 0 0" xyz="0 0 0"/>
+    <parent link="wrist"/>
+    <child link="dummygripper"/>
+    <axis xyz="0 1 0"/>
+    <limit effort="0" lower="0" upper="2" velocity="0"/>
+  </joint>
+  <link name="dummygripper"/>
   <link
     name="i1">
@@ -225,4 +238,5 @@
       effort="0"
       velocity="0" />
+    <mimic joint="gripper"/>
   </joint>
   <link
@@ -283,4 +297,5 @@
       effort="0"
       velocity="0" />
+    <mimic joint="gripper"/>
   </joint>
   <link
@@ -341,4 +356,5 @@
       effort="0"
       velocity="0" />
+    <mimic joint="gripper"/>
   </joint>
   <link
@@ -399,4 +415,5 @@
       effort="0"
       velocity="0" />
+    <mimic joint="gripper"/>
   </joint>
   <link
@@ -457,4 +474,5 @@
       effort="0"
       velocity="0" />
+    <mimic joint="gripper"/>
   </joint>
 </robot>

File: xacro/gummi_ee.srdf.xacro (robot description, xacro)
@@ -8,9 +8,5 @@
   <group name="right_gripper">
     <link name="wrist"/>
-    <joint name="i1f"/>
-    <joint name="i2f"/>
-    <joint name="i3f"/>
-    <joint name="i4f"/>
-    <joint name="i5f"/>
+    <joint name="gripper"/>
   </group>
 </xacro:macro>
