Commit message: Big move over, chnaged files.

File: xacro/gummi_description_ee.urdf.xacro (robot description, xacro)
@@ -1,19 +1,20 @@
 <?xml version="1.0" encoding="utf-8"?>
-<robot>
+<robot
+  name="gummi">
   <link
     name="lowerarm_preroll_d">
     <inertial>
       <origin
-        xyz="0.0192090313803226 -0.000209732444885397 -0.00477606520095217"
-        rpy="0 0 0" />
-      <mass
-        value="0.0573922743530686" />
-      <inertia
-        ixx="5.98272304285402E-07"
-        ixy="-9.55132100709239E-09"
-        ixz="2.00959509125472E-06"
-        iyy="7.34863588332809E-06"
-        iyz="2.84343934345717E-09"
-        izz="6.7503906079721E-06" />
+        xyz="0.0201145573860685 0.000669151743296995 -0.00744229215534365"
+        rpy="0 0 0" />
+      <mass
+        value="0.0734230815881974" />
+      <inertia
+        ixx="1.01515477360727E-05"
+        ixy="4.32433603525769E-08"
+        ixz="7.12477985310256E-06"
+        iyy="1.51518258319088E-05"
+        iyz="-6.16118497879196E-08"
+        izz="5.00102599358937E-06" />
     </inertial>
     <visual>
@@ -41,65 +42,57 @@
     </collision>
   </link>
-  <joint
-    name="fastswitch"
-    type="fixed">
-    <origin
-      xyz="0.056236 -0.019 -0.006"
-      rpy="0 0 0" />
-    <parent
-      link="lowerarm_preroll_u" />
-    <child
+  <joint name="fastswitch" type="fixed">
+    <origin rpy="0 0 0" xyz="0.057 -0.019 -0.005"/>
+    <parent link="lowerarm_preroll_u"/>
+    <child link="lowerarm_preroll_d"/>
+  </joint>
+  <link
+    name="lowerarm">
+    <inertial>
+      <origin
+        xyz="0.0946496953755679 -0.000120356527291464 -0.00129517524906059"
+        rpy="0 0 0" />
+      <mass
+        value="0.181304112038073" />
+      <inertia
+        ixx="5.20535334976771E-05"
+        ixy="1.23954508362984E-06"
+        ixz="-1.5126823036687E-05"
+        iyy="0.000292605338929578"
+        iyz="4.73837407418085E-07"
+        izz="0.000245834375584184" />
+    </inertial>
+    <visual>
+      <origin
+        xyz="0 0 0"
+        rpy="0 0 0" />
+      <geometry>
+        <mesh
+          filename="package://gummi_ee_$(env ROS_GUMMI_EE)/meshes/lowerarm.STL" />
+      </geometry>
+      <material
+        name="">
+        <color
+          rgba="0.792156862745098 0.819607843137255 0.933333333333333 1" />
+      </material>
+    </visual>
+    <collision>
+      <origin
+        xyz="0 0 0"
+        rpy="0 0 0" />
+      <geometry>
+        <mesh
+          filename="package://gummi_ee_$(env ROS_GUMMI_EE)/meshes/lowerarm.STL" />
+      </geometry>
+    </collision>
+  </link>
+  <joint
+    name="forearm_roll"
+    type="revolute">
+    <origin
+      xyz="0.0073346 0.00058424 -0.028344"
+      rpy="0 0 0" />
+    <parent
       link="lowerarm_preroll_d" />
-    <axis
-      xyz="0 0 0" />
-  </joint>
-  <link
-    name="lowerarm">
-    <inertial>
-      <origin
-        xyz="0.076518166900465 0.000154587846369382 0.00668942647768447"
-        rpy="0 0 0" />
-      <mass
-        value="0.214658222402075" />
-      <inertia
-        ixx="2.53797627665925E-05"
-        ixy="-3.78406001691015E-09"
-        ixz="1.36269412886066E-05"
-        iyy="0.000325304336296306"
-        iyz="3.75496083335353E-07"
-        izz="0.000302080494837117" />
-    </inertial>
-    <visual>
-      <origin
-        xyz="0 0 0"
-        rpy="0 0 0" />
-      <geometry>
-        <mesh
-          filename="package://gummi_ee_$(env ROS_GUMMI_EE)/meshes/lowerarm.STL" />
-      </geometry>
-      <material
-        name="">
-        <color
-          rgba="0.792156862745098 0.819607843137255 0.933333333333333 1" />
-      </material>
-    </visual>
-    <collision>
-      <origin
-        xyz="0 0 0"
-        rpy="0 0 0" />
-      <geometry>
-        <mesh
-          filename="package://gummi_ee_$(env ROS_GUMMI_EE)/meshes/lowerarm.STL" />
-      </geometry>
-    </collision>
-  </link>
-  <joint
-    name="forearm_roll"
-    type="continuous">
-    <origin
-      xyz="0.043506 -0.00023376 -0.019876"
-      rpy="0 0 0" />
-    <parent
-      link="lowerarm_preroll_d" />
     <child
       link="lowerarm" />
@@ -107,6 +100,8 @@
       xyz="1 0 0" />
     <limit
-      effort="0"
-      velocity="1" />
+      lower="-1"
+      upper="1"
+      effort="0"
+      velocity="0" />
   </joint>
   <link
@@ -114,15 +109,15 @@
     <inertial>
       <origin
-        xyz="0.0484512742480244 0.0139768664666073 0.000956995637939325"
-        rpy="0 0 0" />
-      <mass
-        value="0.0644774651698934" />
-      <inertia
-        ixx="8.67406414845019E-06"
-        ixy="-1.3193756197629E-05"
-        ixz="-3.41916035169704E-06"
-        iyy="4.217442276821E-05"
-        iyz="-4.04257224014858E-07"
-        izz="4.91399139463636E-05" />
+        xyz="0.0155109020638096 0.0247217069682795 -8.97016135974898E-06"
+        rpy="0 0 0" />
+      <mass
+        value="0.0612417575034934" />
+      <inertia
+        ixx="2.17909064975224E-05"
+        ixy="-1.75146735374738E-07"
+        ixz="7.08623219383127E-09"
+        iyy="1.38582932310292E-05"
+        iyz="4.31485803558046E-11"
+        izz="3.56491921024227E-05" />
     </inertial>
     <visual>
@@ -154,5 +149,5 @@
     type="revolute">
     <origin
-      xyz="0.1511 -0.01935 0.0048471"
+      xyz="0.16463 -0.024 0"
       rpy="0 0 0" />
     <parent
@@ -168,311 +163,714 @@
       velocity="0" />
   </joint>
-  <!--
-  making sure I can move my fingers in a synchronized way. also if they move at
-  different rates, set the mimic tag to something different. it allows for an
-  offset and a multiplication rate. check ros docs for details
-  -->
-  <joint name="gripper" type="revolute">
-    <origin rpy="0 0 0" xyz="0 0 0"/>
-    <parent link="wrist"/>
-    <child link="dummygripper"/>
-    <axis xyz="0 1 0"/>
-    <limit effort="0" lower="0" upper="2" velocity="0"/>
-  </joint>
-  <link name="dummygripper"/>
-  <link
-    name="i1">
-    <inertial>
-      <origin
-        xyz="0.0230748926267925 0.00588066789200992 0.00129219082652174"
-        rpy="0 0 0" />
-      <mass
-        value="0.00632408233084942" />
-      <inertia
-        ixx="3.56498343502738E-08"
-        ixy="-7.51978011656011E-09"
-        ixz="7.65091950170785E-08"
-        iyy="1.38099634070148E-06"
-        iyz="2.95085409823962E-09"
-        izz="1.34584197546666E-06" />
-    </inertial>
-    <visual>
-      <origin
-        xyz="0 0 0"
-        rpy="0 0 0" />
-      <geometry>
-        <mesh
-          filename="package://gummi_ee_$(env ROS_GUMMI_EE)/meshes/i1.STL" />
-      </geometry>
-      <material
-        name="">
-        <color
-          rgba="0.792156862745098 0.819607843137255 0.933333333333333 1" />
-      </material>
-    </visual>
-    <collision>
-      <origin
-        xyz="0 0 0"
-        rpy="0 0 0" />
-      <geometry>
-        <mesh
-          filename="package://gummi_ee_$(env ROS_GUMMI_EE)/meshes/i1.STL" />
-      </geometry>
-    </collision>
-  </link>
-  <joint
-    name="i1f"
+  <link
+    name="gbase">
+    <inertial>
+      <origin
+        xyz="0.0375396345255545 0.000258621653510823 0.000308025751646932"
+        rpy="0 0 0" />
+      <mass
+        value="0.112572451212744" />
+      <inertia
+        ixx="3.46149816301849E-08"
+        ixy="3.71824830981742E-07"
+        ixz="-8.88625729821223E-07"
+        iyy="5.74238369795189E-05"
+        iyz="8.8502104967547E-09"
+        izz="5.74191745262333E-05" />
+    </inertial>
+    <visual>
+      <origin
+        xyz="0 0 0"
+        rpy="0 0 0" />
+      <geometry>
+        <mesh
+          filename="package://gummi_ee_$(env ROS_GUMMI_EE)/meshes/gbase.STL" />
+      </geometry>
+      <material
+        name="">
+        <color
+          rgba="0.792156862745098 0.819607843137255 0.933333333333333 1" />
+      </material>
+    </visual>
+    <collision>
+      <origin
+        xyz="0 0 0"
+        rpy="0 0 0" />
+      <geometry>
+        <mesh
+          filename="package://gummi_ee_$(env ROS_GUMMI_EE)/meshes/gbase.STL" />
+      </geometry>
+    </collision>
+  </link>
+  <joint
+    name="gdovetail"
+    type="fixed">
+    <origin
+      xyz="0.043 0.02425 0"
+      rpy="0 0 0" />
+    <parent
+      link="wrist" />
+    <child
+      link="gbase" />
+    <axis
+      xyz="0 0 0" />
+  </joint>
+  <link
+    name="g_camera">
+    <inertial>
+      <origin
+        xyz="-0.0130038062547488 0.000414347997380345 -0.00115139779329799"
+        rpy="0 0 0" />
+      <mass
+        value="0.0054126706518889" />
+      <inertia
+        ixx="0"
+        ixy="0"
+        ixz="0"
+        iyy="0"
+        iyz="0"
+        izz="0" />
+    </inertial>
+    <visual>
+      <origin
+        xyz="0 0 0"
+        rpy="0 0 0" />
+      <geometry>
+        <mesh
+          filename="package://gummi_ee_$(env ROS_GUMMI_EE)/meshes/g_camera.STL" />
+      </geometry>
+      <material
+        name="">
+        <color
+          rgba="0.792156862745098 0.819607843137255 0.933333333333333 1" />
+      </material>
+    </visual>
+    <collision>
+      <origin
+        xyz="0 0 0"
+        rpy="0 0 0" />
+      <geometry>
+        <mesh
+          filename="package://gummi_ee_$(env ROS_GUMMI_EE)/meshes/g_camera.STL" />
+      </geometry>
+    </collision>
+  </link>
+  <joint
+    name="g_c_j"
+    type="fixed">
+    <origin
+      xyz="0.078543 5.1126E-05 0.00058816"
+      rpy="0 0 0" />
+    <parent
+      link="gbase" />
+    <child
+      link="g_camera" />
+    <axis
+      xyz="0 0 0" />
+  </joint>
+  <link
+    name="g_um">
+    <inertial>
+      <origin
+        xyz="0.00245238145288562 -0.0217265687128561 -0.0105911469473412"
+        rpy="0 0 0" />
+      <mass
+        value="0.0108804943967655" />
+      <inertia
+        ixx="8.08735422601889E-08"
+        ixy="4.97110946899304E-08"
+        ixz="-1.39273928121627E-09"
+        iyy="4.53539384016324E-08"
+        iyz="6.17358200741367E-10"
+        izz="1.26078407713655E-07" />
+    </inertial>
+    <visual>
+      <origin
+        xyz="0 0 0"
+        rpy="0 0 0" />
+      <geometry>
+        <mesh
+          filename="package://gummi_ee_$(env ROS_GUMMI_EE)/meshes/g_um.STL" />
+      </geometry>
+      <material
+        name="">
+        <color
+          rgba="0.792156862745098 0.819607843137255 0.933333333333333 1" />
+      </material>
+    </visual>
+    <collision>
+      <origin
+        xyz="0 0 0"
+        rpy="0 0 0" />
+      <geometry>
+        <mesh
+          filename="package://gummi_ee_$(env ROS_GUMMI_EE)/meshes/g_um.STL" />
+      </geometry>
+    </collision>
+  </link>
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
File: xacro/gummi_ee.srdf.xacro (robot description, xacro)
@@ -4,8 +4,11 @@
     <joint name="forearm_roll" />
     <joint name="wrist_pitch" />
+    <joint name="coupling_tool"/>
+    <joint name="gdovetail"/>
 </xacro:macro>
 <xacro:macro name="group_right_gripper_ee">
   <group name="right_gripper">
     <link name="wrist"/>
+    <link name="gbase"/>
     <joint name="gripper"/>
   </group>
@@ -17,32 +20,30 @@
 <xacro:macro name="end_effector_ee">
   <!--END EFFECTOR: Purpose: Represent information about an end effector.-->
-<end_effector group="right_gripper" name="right_eef" parent_link="wrist" parent_group="right_arm"/>
+<end_effector group="right_gripper" name="right_eef" parent_link="tool" parent_group="right_arm"/>
 </xacro:macro>
 <xacro:macro name="disable_collisions_ee">
-  <!-- <disable_collisions link1="right_hand" link2="wrist" reason="Never" />
-  <disable_collisions link1="right_hand" link2="gripper_link" reason="Never" /> -->
-  <disable_collisions link1="i1" link2="lowerarm" reason="Never" />
-  <disable_collisions link1="i2" link2="lowerarm" reason="Never" />
-  <disable_collisions link1="i3" link2="lowerarm" reason="Never" />
-  <disable_collisions link1="i4" link2="lowerarm" reason="Never" />
-  <disable_collisions link1="i5" link2="lowerarm" reason="Never" />
-  <disable_collisions link1="i1" link2="wrist" reason="Never" />
-  <disable_collisions link1="i2" link2="wrist" reason="Never" />
-  <disable_collisions link1="i3" link2="wrist" reason="Never" />
-  <disable_collisions link1="i4" link2="wrist" reason="Never" />
-  <disable_collisions link1="i5" link2="wrist" reason="Never" />
-  <disable_collisions link1="i1" link2="i2" reason="Never" />
-  <disable_collisions link1="i1" link2="i3" reason="Never" />
-  <disable_collisions link1="i1" link2="i4" reason="Never" />
-  <disable_collisions link1="i1" link2="i5" reason="Never" />
-  <disable_collisions link1="i2" link2="i3" reason="Never" />
-  <disable_collisions link1="i2" link2="i4" reason="Never" />
-  <disable_collisions link1="i2" link2="i5" reason="Never" />
-  <disable_collisions link1="i3" link2="i4" reason="Never" />
-  <disable_collisions link1="i3" link2="i5" reason="Never" />
-  <disable_collisions link1="i4" link2="i5" reason="Never" />
+  <disable_collisions link1="tool" link2="wrist" reason="Adjacent" />
   <disable_collisions link1="lowerarm" link2="lowerarm_preroll_d" reason="Adjacent" />
   <disable_collisions link1="lowerarm" link2="wrist" reason="Adjacent" />
   <disable_collisions link1="lowerarm_preroll_d" link2="wrist" reason="Never" />
+  <disable_collisions link1="lowerarm" link2="wrist_ext_pulley" reason="Adjacent"/>
+  <disable_collisions link1="lowerarm" link2="wrist_flex_pulley" reason="Adjacent"/>
+  <!-- gripper collisions  -->
+  <disable_collisions link1="gbase" link2="wrist" reason="Adjacent"/>
+  <disable_collisions link1="gbase" link2="g_camera" reason="Adjacent"/>
+  <disable_collisions link1="gbase" link2="g_um" reason="Adjacent"/>
+  <disable_collisions link1="gbase" link2="g_ll" reason="Adjacent"/>
+  <disable_collisions link1="gbase" link2="g_ug" reason="Adjacent"/>
+  <disable_collisions link1="gbase" link2="g_lg" reason="Adjacent"/>
+  <disable_collisions link1="gbase" link2="g_mfl" reason="Adjacent"/>
+  <disable_collisions link1="gbase" link2="g_lfl" reason="Adjacent"/>
+  <disable_collisions link1="gbase" link2="g_mf" reason="Never"/>
+  <disable_collisions link1="gbase" link2="g_lf" reason="Never"/>
+  <disable_collisions link1="g_ug" link2="g_um" reason="Adjacent"/>
+  <disable_collisions link1="g_lg" link2="g_ll" reason="Adjacent"/>
+  <disable_collisions link1="g_lf" link2="g_um" reason="Adjacent"/>
+  <disable_collisions link1="g_mf" link2="g_ll" reason="Adjacent"/>
+  <disable_collisions link1="g_lf" link2="g_lfl" reason="Adjacent"/>
+  <disable_collisions link1="g_mf" link2="g_mfl" reason="Adjacent"/>
 </xacro:macro>
 </robot>

Commit message: Without forearm_roll moving ok, not moveit yet.

File: xacro/gummi_description_ee.urdf.xacro (robot description, xacro)
@@ -89,5 +89,5 @@
   <joint
     name="forearm_roll"
-    type="revolute">
+    type="fixed">
     <origin
       xyz="0.0073346 0.00058424 -0.028344"

File: xacro/gummi_ee.srdf.xacro (robot description, xacro)
@@ -2,5 +2,4 @@
 <robot name="gummi" xmlns:xacro="http://www.ros.org/wiki/xacro">
 <xacro:macro name="group_right_arm_ee">
-    <joint name="forearm_roll" />
     <joint name="wrist_pitch" />
     <joint name="coupling_tool"/>
@@ -15,5 +14,4 @@
 </xacro:macro>
 <xacro:macro name="group_state_right_arm_ee">
-  <joint name="forearm_roll" value="0" />
   <joint name="wrist_pitch" value="0" />
 </xacro:macro>

Commit message: Working with forearm_roll back.

File: xacro/gummi_description_ee.urdf.xacro (robot description, xacro)
@@ -89,5 +89,5 @@
   <joint
     name="forearm_roll"
-    type="fixed">
+    type="revolute">
     <origin
       xyz="0.0073346 0.00058424 -0.028344"
@@ -156,7 +156,7 @@
       link="wrist" />
     <axis
-      xyz="0 1 0" />
-    <limit
-      lower="-1"
+      xyz="0 -1 0" />
+    <limit
+      lower="-0.6"
       upper="1"
       effort="0"

File: xacro/gummi_ee.srdf.xacro (robot description, xacro)
@@ -2,4 +2,5 @@
 <robot name="gummi" xmlns:xacro="http://www.ros.org/wiki/xacro">
 <xacro:macro name="group_right_arm_ee">
+    <joint name="forearm_roll" />
     <joint name="wrist_pitch" />
     <joint name="coupling_tool"/>
@@ -14,4 +15,5 @@
 </xacro:macro>
 <xacro:macro name="group_state_right_arm_ee">
+  <joint name="forearm_roll" value="0" />
   <joint name="wrist_pitch" value="0" />
 </xacro:macro>
